Commit message: Update Sirius wheel stand

File: source/robot_lab/data/Robots/CUHKLRL/Sirius_wheel/Sirius_Wheel_description/urdf/sirius_wheel.urdf (robot description, URDF)
Before this commit: robot Sirius_Wheel_description, 22 links, 21 joints
Links:
- added link base
Joints:
- added joint base_joint: type fixed, parent base, child trunk, origin xyz=0 0 0 rpy=0 -1.57 0
